Commit message: Organize file structure into robot and world

File: src/lazershark_sim/robot/lazershark_sim.urdf (robot description, URDF)
Before this commit: robot lazershark_sim, 12 links, 11 joints
Links:
- link base_link: geometry collision mesh filename=package://lazershark_sim/robot/meshes/base_link.STL; visual mesh filename=package://lazershark_sim/robot/meshes/base_link.STL
- link dvl_link: geometry collision mesh filename=package://lazershark_sim/robot/meshes/dvl_link.STL; visual mesh filename=package://lazershark_sim/robot/meshes/dvl_link.STL
- link imu_link: geometry collision mesh filename=package://lazershark_sim/robot/meshes/imu_link.STL; visual mesh filename=package://lazershark_sim/robot/meshes/imu_link.STL
- link thruster_0: geometry collision mesh filename=package://lazershark_sim/robot/meshes/thruster_0.STL; visual mesh filename=package://lazershark_sim/robot/meshes/thruster_0.STL
- link thruster_1: geometry collision mesh filename=package://lazershark_sim/robot/meshes/thruster_1.STL; visual mesh filename=package://lazershark_sim/robot/meshes/thruster_1.STL
- link thruster_2: geometry collision mesh filename=package://lazershark_sim/robot/meshes/thruster_2.STL; visual mesh filename=package://lazershark_sim/robot/meshes/thruster_2.STL
- link thruster_3: geometry collision mesh filename=package://lazershark_sim/robot/meshes/thruster_3.STL; visual mesh filename=package://lazershark_sim/robot/meshes/thruster_3.STL
- link thruster_4: geometry collision mesh filename=package://lazershark_sim/robot/meshes/thruster_4.STL; visual mesh filename=package://lazershark_sim/robot/meshes/thruster_4.STL
- link thruster_5: geometry collision mesh filename=package://lazershark_sim/robot/meshes/thruster_5.STL; visual mesh filename=package://lazershark_sim/robot/meshes/thruster_5.STL
- link thruster_6: geometry collision mesh filename=package://lazershark_sim/robot/meshes/thruster_6.STL; visual mesh filename=package://lazershark_sim/robot/meshes/thruster_6.STL
- link thruster_7: geometry collision mesh filename=package://lazershark_sim/robot/meshes/thruster_7.STL; visual mesh filename=package://lazershark_sim/robot/meshes/thruster_7.STL
- link zed_camera_link: geometry collision mesh filename=package://lazershark_sim/robot/meshes/zed_camera_link.STL; visual mesh filename=package://lazershark_sim/robot/meshes/zed_camera_link.STL

Commit message: removed collisions

File: src/lazershark_sim/robot/lazershark_sim.urdf (robot description, URDF)
Before this commit: robot lazershark_sim, 12 links, 11 joints
Links:
- link base_link: geometry visual mesh filename=package://lazershark_sim/robot/meshes/base_link.STL
- link dvl_link: geometry visual mesh filename=package://lazershark_sim/robot/meshes/dvl_link.STL
- link imu_link: geometry visual mesh filename=package://lazershark_sim/robot/meshes/imu_link.STL
- link thruster_0: geometry visual mesh filename=package://lazershark_sim/robot/meshes/thruster_0.STL
- link thruster_1: geometry visual mesh filename=package://lazershark_sim/robot/meshes/thruster_1.STL
- link thruster_2: geometry visual mesh filename=package://lazershark_sim/robot/meshes/thruster_2.STL
- link thruster_3: geometry visual mesh filename=package://lazershark_sim/robot/meshes/thruster_3.STL
- link thruster_4: geometry visual mesh filename=package://lazershark_sim/robot/meshes/thruster_4.STL
- link thruster_5: geometry visual mesh filename=package://lazershark_sim/robot/meshes/thruster_5.STL
- link thruster_6: geometry visual mesh filename=package://lazershark_sim/robot/meshes/thruster_6.STL
- link thruster_7: geometry visual mesh filename=package://lazershark_sim/robot/meshes/thruster_7.STL
- link zed_camera_link: geometry visual mesh filename=package://lazershark_sim/robot/meshes/zed_camera_link.STL

Commit message: new urdf with material properties

File: src/lazershark_sim/robot/lazershark_sim.urdf (robot description, URDF)
Before this commit: robot lazershark_sim, 12 links, 11 joints
Links:
- link base_link: mass 5.76928449442786 -> 15.577; geometry collision mesh filename=package://lazershark_sim/robot/meshes/base_link.STL; visual mesh filename=package://lazershark_sim/robot/meshes/base_link.STL
- link dvl_link: mass 0.25634 -> 0.25633622835366; geometry collision mesh filename=package://lazershark_sim/robot/meshes/dvl_link.STL; visual mesh filename=package://lazershark_sim/robot/meshes/dvl_link.STL
- link imu_link: geometry collision mesh filename=package://lazershark_sim/robot/meshes/imu_link.STL; visual mesh filename=package://lazershark_sim/robot/meshes/imu_link.STL
- link thruster_0: mass 0.0077410181298602 -> 0.007741; geometry collision mesh filename=package://lazershark_sim/robot/meshes/thruster_0.STL; visual mesh filename=package://lazershark_sim/robot/meshes/thruster_0.STL
- link thruster_1: mass 0.0077421 -> 0.00774208667120841; geometry collision mesh filename=package://lazershark_sim/robot/meshes/thruster_1.STL; visual mesh filename=package://lazershark_sim/robot/meshes/thruster_1.STL
- link thruster_2: mass 0.00774117141861991 -> 0.00774117302951113; geometry collision mesh filename=package://lazershark_sim/robot/meshes/thruster_2.STL; visual mesh filename=package://lazershark_sim/robot/meshes/thruster_2.STL
- link thruster_3: geometry collision mesh filename=package://lazershark_sim/robot/meshes/thruster_3.STL; visual mesh filename=package://lazershark_sim/robot/meshes/thruster_3.STL
- link thruster_4: mass 0.00773999758129765 -> 0.00773999910275849; geometry collision mesh filename=package://lazershark_sim/robot/meshes/thruster_4.STL; visual mesh filename=package://lazershark_sim/robot/meshes/thruster_4.STL
- link thruster_5: geometry collision mesh filename=package://lazershark_sim/robot/meshes/thruster_5.STL; visual mesh filename=package://lazershark_sim/robot/meshes/thruster_5.STL
- link thruster_6: mass 0.00773999839485437 -> 0.00773999910275899; geometry collision mesh filename=package://lazershark_sim/robot/meshes/thruster_6.STL; visual mesh filename=package://lazershark_sim/robot/meshes/thruster_6.STL
- link thruster_7: mass 0.00773999925817228 -> 0.00773999839485365; geometry collision mesh filename=package://lazershark_sim/robot/meshes/thruster_7.STL; visual mesh filename=package://lazershark_sim/robot/meshes/thruster_7.STL
- link zed_camera_link: geometry collision mesh filename=package://lazershark_sim/robot/meshes/zed_camera_link.STL; visual mesh filename=package://lazershark_sim/robot/meshes/zed_camera_link.STL
Joints:
- joint thruster_joint_0: limit lower=0 upper=30 effort=5 velocity=5 -> lower=-1000000000000 upper=1000000000000 effort=-1 velocity=-1
- joint thruster_joint_1: axis -0.707106781186549 0.707106781186546 0 -> -0.70711 0.70711 0; limit lower=0 upper=30 effort=5 velocity=5 -> lower=-1000000000000 upper=1000000000000 effort=-1 velocity=-1
- joint thruster_joint_2: axis -0.707106781186544 -0.707106781186551 0 -> -0.70711 -0.70711 0; limit lower=0 upper=30 effort=5 velocity=5 -> lower=-1000000000000 upper=1000000000000 effort=-1 velocity=-1
- joint thruster_joint_3: axis 0.707106781186551 -0.707106781186544 0 -> 0.70711 -0.70711 0; limit lower=0 upper=30 effort=5 velocity=5 -> lower=-1000000000000 upper=1000000000000 effort=-1 velocity=-1
- joint thruster_joint_4: limit lower=0 upper=30 effort=5 velocity=5 -> lower=-1000000000000 upper=1000000000000 effort=-1 velocity=-1
- joint thruster_joint_5: limit lower=0 upper=30 effort=5 velocity=5 -> lower=-1000000000000 upper=1000000000000 effort=-1 velocity=-1
- joint thruster_joint_6: limit lower=0 upper=30 effort=5 velocity=5 -> lower=-1000000000000 upper=1000000000000 effort=-1 velocity=-1
- joint thruster_joint_7: limit lower=0 upper=30 effort=5 velocity=5 -> lower=-1000000000000 upper=1000000000000 effort=-1 velocity=-1
