Commit message: Made required changes to SDF

File: src/lazershark/lazershark_sim/robot/lazershark_sim.urdf (robot description, URDF)
Before this commit: robot lazershark_sim, 12 links, 11 joints
Links:
- removed link dvl_link
- removed link imu_link
- removed link thruster_0
- removed link thruster_1
- removed link thruster_2
- removed link thruster_3
- removed link thruster_5
- removed link thruster_6
- removed link thruster_7
- removed link zed_camera_link
- added link camera_zed, mass 0.152258681193599; collision mesh filename=package://lazershark_sim/robot/meshes/camera_zed.STL; visual mesh filename=package://lazershark_sim/robot/meshes/camera_zed.STL
- added link dvl_a50, mass 0.25633622835366; collision mesh filename=package://lazershark_sim/robot/meshes/dvl_a50.STL; visual mesh filename=package://lazershark_sim/robot/meshes/dvl_a50.STL
- added link imu_naviguider0, mass 0.00104001214902657; collision mesh filename=package://lazershark_sim/robot/meshes/imu_naviguider0.STL; visual mesh filename=package://lazershark_sim/robot/meshes/imu_naviguider0.STL
- added link imu_naviguider1, mass 0.00104001214902657; collision mesh filename=package://lazershark_sim/robot/meshes/imu_naviguider1.STL; visual mesh filename=package://lazershark_sim/robot/meshes/imu_naviguider1.STL
- added link imu_targetpoint0, mass 0.00550725674074068; collision mesh filename=package://lazershark_sim/robot/meshes/imu_targetpoint0.STL; visual mesh filename=package://lazershark_sim/robot/meshes/imu_targetpoint0.STL
- added link imu_targetpoint1, mass 0.00550725674074067; collision mesh filename=package://lazershark_sim/robot/meshes/imu_targetpoint1.STL; visual mesh filename=package://lazershark_sim/robot/meshes/imu_targetpoint1.STL
- added link thruster0, mass 0.00774021849814979; collision mesh filename=package://lazershark_sim/robot/meshes/thruster0.STL; visual mesh filename=package://lazershark_sim/robot/meshes/thruster0.STL
- added link thruster1, mass 0.00773999910275849; collision mesh filename=package://lazershark_sim/robot/meshes/thruster1.STL; visual mesh filename=package://lazershark_sim/robot/meshes/thruster1.STL
- added link thruster2, mass 0.00773999910275899; collision mesh filename=package://lazershark_sim/robot/meshes/thruster2.STL; visual mesh filename=package://lazershark_sim/robot/meshes/thruster2.STL
- added link thruster3, mass 0.00773999839485365; collision mesh filename=package://lazershark_sim/robot/meshes/thruster3.STL; visual mesh filename=package://lazershark_sim/robot/meshes/thruster3.STL
- added link thruster5, mass 0.00774117302951113; collision mesh filename=package://lazershark_sim/robot/meshes/thruster5.STL; visual mesh filename=package://lazershark_sim/robot/meshes/thruster5.STL
- added link thruster6, mass 0.00774208667120787; collision mesh filename=package://lazershark_sim/robot/meshes/thruster6.STL; visual mesh filename=package://lazershark_sim/robot/meshes/thruster6.STL
- added link thruster7, mass 0.00774152572047315; collision mesh filename=package://lazershark_sim/robot/meshes/thruster7.STL; visual mesh filename=package://lazershark_sim/robot/meshes/thruster7.STL
- link base_link: mass 15.577 -> 15.9199897324527
- link thruster_4: mass 0.00773999910275849 -> 0.00774122350372358
Joints:
- removed joint imu_joint
- removed joint zed_camera_joint
- added joint camera_zed_joint: type fixed, parent base_link, child camera_zed, origin xyz=0 0 0 rpy=0 0 0, axis 0 0 0, limit lower=0 upper=0 effort=0 velocity=0
- added joint imu_naviguider0_joint: type fixed, parent base_link, child imu_naviguider0, origin xyz=0 0 0 rpy=0 0 0, axis 0 0 0
- added joint imu_naviguider1_joint: type fixed, parent base_link, child imu_naviguider1, origin xyz=0 0 0 rpy=0 0 0, axis 0 0 0
- added joint imu_targetpoint0_joint: type fixed, parent base_link, child imu_targetpoint0, origin xyz=0 0 0 rpy=0 0 0, axis 0 0 0
- added joint imu_targetpoint1_joint: type fixed, parent base_link, child imu_targetpoint1, origin xyz=0 0 0 rpy=0 0 0, axis 0 0 0
- joint dvl_joint: child dvl_link -> dvl_a50
- joint thruster_joint_0: child thruster_0 -> thruster0
- joint thruster_joint_1: axis -0.70711 0.70711 0 -> 0 0 -1; child thruster_1 -> thruster1
- joint thruster_joint_2: axis -0.70711 -0.70711 0 -> 0 0 -1; child thruster_2 -> thruster2
- joint thruster_joint_3: axis 0.70711 -0.70711 0 -> 0 0 -1; child thruster_3 -> thruster3; type continuous -> revolute
- joint thruster_joint_4: axis 0 0 -1 -> -0.707106781186552 0.707106781186543 0
- joint thruster_joint_5: axis 0.70711 0.70711 0 -> -0.707106781186544 -0.707106781186551 0; child thruster_5 -> thruster5
- joint thruster_joint_6: axis 0 0 -1 -> 0.707106781186551 -0.707106781186544 0; child thruster_6 -> thruster6; type revolute -> continuous
- joint thruster_joint_7: axis 0 0 -1 -> 0.707106781186544 0.707106781186551 0; child thruster_7 -> thruster7
