Commit message: SDF including transforms for sensors -- FIX DIRECTIONS

File: src/lazershark/sim/robot/lazershark_sim.urdf (robot description, URDF)
Before this commit: robot lazershark_sim, 15 links, 14 joints
Links:
- link base_link: mass 15.9199897324527 -> 15.9199897349552; geometry collision mesh filename=package://urdf_export_5/meshes/base_link.STL; visual mesh filename=package://urdf_export_5/meshes/base_link.STL
- link camera_zed: mass 0.152258681193599 -> 0.152258681193596; geometry collision mesh filename=package://urdf_export_5/meshes/camera_zed.STL; visual mesh filename=package://urdf_export_5/meshes/camera_zed.STL
- link dvl_a50: geometry collision mesh filename=package://urdf_export_5/meshes/dvl_a50.STL; visual mesh filename=package://urdf_export_5/meshes/dvl_a50.STL
- link imu_naviguider0: geometry collision mesh filename=package://urdf_export_5/meshes/imu_naviguider0.STL; visual mesh filename=package://urdf_export_5/meshes/imu_naviguider0.STL
- link imu_naviguider1: geometry collision mesh filename=package://urdf_export_5/meshes/imu_naviguider1.STL; visual mesh filename=package://urdf_export_5/meshes/imu_naviguider1.STL
- link imu_targetpoint0: geometry collision mesh filename=package://urdf_export_5/meshes/imu_targetpoint0.STL; visual mesh filename=package://urdf_export_5/meshes/imu_targetpoint0.STL
- link imu_targetpoint1: geometry collision mesh filename=package://urdf_export_5/meshes/imu_targetpoint1.STL; visual mesh filename=package://urdf_export_5/meshes/imu_targetpoint1.STL
- link thruster0: geometry collision mesh filename=package://urdf_export_5/meshes/thruster0.STL; visual mesh filename=package://urdf_export_5/meshes/thruster0.STL
- link thruster1: geometry collision mesh filename=package://urdf_export_5/meshes/thruster1.STL; visual mesh filename=package://urdf_export_5/meshes/thruster1.STL
- link thruster2: geometry collision mesh filename=package://urdf_export_5/meshes/thruster2.STL; visual mesh filename=package://urdf_export_5/meshes/thruster2.STL
- link thruster3: geometry collision mesh filename=package://urdf_export_5/meshes/thruster3.STL; visual mesh filename=package://urdf_export_5/meshes/thruster3.STL
- link thruster5: geometry collision mesh filename=package://urdf_export_5/meshes/thruster5.STL; visual mesh filename=package://urdf_export_5/meshes/thruster5.STL
- link thruster6: geometry collision mesh filename=package://urdf_export_5/meshes/thruster6.STL; visual mesh filename=package://urdf_export_5/meshes/thruster6.STL
- link thruster7: geometry collision mesh filename=package://urdf_export_5/meshes/thruster7.STL; visual mesh filename=package://urdf_export_5/meshes/thruster7.STL
- link thruster_4: geometry collision mesh filename=package://urdf_export_5/meshes/thruster_4.STL; visual mesh filename=package://urdf_export_5/meshes/thruster_4.STL
